File: ForgeX/BlackDev_G0Basic/BlackDev_G0Basic.kicad_sch (KiCad schematic)
At the start: 10 parts, among them J1 Conn_01x02_Pin, J6 Conn_02x20_Odd_Even

Commit message: BlackDevG0 Basic communication update
Added Esp32 as an SPI slave allowing for Telemetry, CAN (TWAI) connection , TCP/IP - UDP Logging, SD-CARD based logging, for a seamless R&D experience
Parts:
- removed R5: 22, Resistor_SMD:R_0603_1608Metric_Pad0.98x0.95mm_HandSolder, symbol Device:R
- added C1, C2: 10u, Capacitor_SMD:C_1206_3216Metric_Pad1.33x1.80mm_HandSolder, symbol Device:C
- added C3: 100n, Capacitor_SMD:C_0603_1608Metric_Pad1.08x0.95mm_HandSolder, symbol Device:C
- added C4, C5: 1u, Capacitor_SMD:C_0603_1608Metric_Pad1.08x0.95mm_HandSolder, symbol Device:C
- added J2: PROG, Connector_PinHeader_2.54mm:PinHeader_1x05_P2.54mm_Vertical_SMD_Pin1Left, symbol Connector:Conn_01x05_Pin
- added J3: Conn_01x02_Pin, Connector_PinHeader_2.54mm:PinHeader_1x02_P2.54mm_Vertical, symbol Connector:Conn_01x02_Pin
- added J4: Conn_01x04_Pin, Connector_JST:JST_XH_B4B-XH-A_1x04_P2.50mm_Vertical, symbol Connector:Conn_01x04_Pin
- added R10: 120, Resistor_SMD:R_1206_3216Metric_Pad1.30x1.75mm_HandSolder, symbol Device:R
- added R11, R9: 10k, Capacitor_SMD:C_0603_1608Metric_Pad1.08x0.95mm_HandSolder, symbol Device:R
- added R12: 22, Resistor_SMD:R_0603_1608Metric_Pad0.98x0.95mm_HandSolder, symbol Device:R
- added U2: ESP32-WROOM-32E, EasyEDA:WIFI-SMD_ESP32-WROOM-32E, symbol EasyEDA:ESP32-WROOM-32E
- added U3: AMS1117-3.3, Package_TO_SOT_SMD:SOT-223-3_TabPin2, symbol Regulator_Linear:AMS1117-3.3
- added U4: SIT65HVD230DR, EasyEDA:SOP-8_L4.9-W3.9-P1.27-LS6.0-BL, symbol EasyEDA:SIT65HVD230DR
- added U5: HX TF PUSH, EasyEDA:TF-SMD_TF-PUSH, symbol EasyEDA:HXTFPUSH
- J1: footprint Connector_PinHeader_2.54mm:PinHeader_1x02_P2.54mm_Vertical -> Connector_PinHeader_2.54mm:PinHeader_1x02_P2.54mm_Vertical_SMD_Pin1Right
Connections:
- net 5V: now also C2.1, U3.3 (VI)
- net EXP_CS2: now also U2.31 (IO19)
- net EXP_MISO: now also U1.12 (PB4), R12.2
- net EXP_MOSI: now also U2.28 (IO17)
- net EXP_SCLK: now also U2.27 (IO16)
- net GND: now also C1.2, C2.2, C3.2, C4.2, C5.2, J2.1 (Pin_1), J4.3 (Pin_3), J4.4 (Pin_4), R11.1, U2.1 (GND), U2.15 (GND), U2.38 (GND), U2.39 (GND), U3.1 (GND), U4.2 (GND), U5.10 (SHELL), U5.11 (SHELL), U5.12 (SHELL), U5.13 (SHELL), U5.6 (VSS)
- net ESP_IRQ: now reaches U1.36 (PB2)
- net ESP_IRQ: now also U2.33 (IO21)
- new net: R12.1, U2.30 (IO18)
- new net: J2.5 (Pin_5), U2.34 (RXD0)
- new net: J2.4 (Pin_4), U2.35 (TXD0)
- new net: J3.2 (Pin_2), R10.2
- new net: R11.2, U4.8 (RS)
- new net 3.3V: C1.1, C3.1, C4.1, C5.1, R9.2, U2.2 (3V3), U3.2 (VO), U4.3 (VCC), U5.4 (VDD)
- new net Boot0: J2.3 (Pin_3), U2.25 (IO0)
- new net CANH: J3.1 (Pin_1), J4.1 (Pin_1), U4.7 (CANH)
- new net CANL: J4.2 (Pin_2), R10.1, U4.6 (CANL)
- new net CAN_RXD: U2.37 (IO23), U4.4 (R)
- new net CAN_TXD: U2.36 (IO22), U4.1 (D)
- new net ESP_RST: J2.2 (Pin_2), R9.1, U2.3 (EN)
- new net SD_CLK: U2.13 (IO14), U5.5 (CLK)
- new net SD_CMD: U2.23 (IO15), U5.3 (CMD)
- new net SD_DAT0: U2.24 (IO2), U5.7 (DAT0)
- new net SD_DAT1: U2.26 (IO4), U5.8 (DAT1)
- new net SD_DAT2: U2.14 (IO12), U5.1 (DAT2)
- new net SD_DAT3: U2.16 (IO13), U5.2 (CD/DAT3)
- no-connect marks 10 -> 28
Other:
- moved on the sheet: J1, J6, R1, R2, R3, R4, R6, R7, U1
