File: ForgeX/LVP_G0S4B/revA/LVP_G0S4B.kicad_pcb (KiCad board)
At the start: 2 copper layers, 159.9 x 47.5 mm, 61 parts, among them J1 Conn_02x05_Odd_Even, J11 Conn_01x02_Pin, J12 Conn_01x02_Pin, J13 Conn_01x02_Pin, J14 Conn_02x05_Odd_Even, J15 Conn_01x02_Pin, J16 Conn_01x04, J17 Conn_01x04, J2 Conn_02x05_Odd_Even, J3 Conn_02x05_Odd_Even, J4 Conn_02x05_Odd_Even, J5 Conn_01x06_Pin, J6 Conn_02x20_Odd_Even, J7 Conn_01x02_Pin, J8 Conn_01x02_Pin, J9 Conn_01x03_Pin, Q2 AO3400A, U4 AMS1117-3.3

Commit message: PMB low voltage variant
Low voltage PMB variant up to 80V,  with SEM mark
Other:
- board text added: "SEM"
