File: ForgeX/PMB_G0S4V80B/revA/PMB_G0S4V80B.kicad_pcb (KiCad board)
At the start: 2 copper layers, 160.1 x 45.1 mm, 22 parts, among them J1 Screw_Terminal_01x03, J12 Screw_Terminal_01x03, J13 Screw_Terminal_01x01, J14 Screw_Terminal_01x01, J17 Screw_Terminal_01x01, J2 Screw_Terminal_01x03, J3 Screw_Terminal_01x03, J4 Screw_Terminal_01x01, J5 Screw_Terminal_01x01, J6 Screw_Terminal_01x01, J8 Screw_Terminal_01x01, J9 Screw_Terminal_01x01

Commit message: PMB_G0SV80B finale
Parts:
- added D1: P6KE47A, Diode_THT:D_DO-15_P10.16mm_Horizontal, F.Cu at (236.1, 47.1)
